File: kicad/LixieMounter/LixieMounter.kicad_pcb (KiCad board)
At the start: 2 copper layers, 100 x 50 mm, 5 parts, among them J1 Conn_01x06, J2 Conn_01x10, U1 2DigitLixie, U2 2DigitLixie, U3 2DigitLixie

Commit message: 暫定的な基板の完成
Other:
- net class Default: trace_width 0.75 -> 1
